File: WS_Wheel_PCB.kicad_pcb (KiCad board)
At the start: 2 copper layers, 6 parts, among them U1 Teensy4.1

Commit message: Saving for the day
Parts:
- removed MAX1: ~, Custom_Components:MAX3002
- added C1: ~, Connector_Molex:Molex_Nano-Fit_105310-xx12_2x06_P2.50mm_Vertical, F.Cu at (132.0, 47.0)
- added C2: ~, Connector_Molex:Molex_Nano-Fit_105310-xx12_2x06_P2.50mm_Vertical, F.Cu at (177.0, 47.0)
- added C3: ~, Connector_Molex:Molex_Nano-Fit_105310-xx12_2x06_P2.50mm_Vertical, F.Cu at (119.0, 77.0)
- added C4: ~, Connector_Molex:Molex_Nano-Fit_105310-xx12_2x06_P2.50mm_Vertical, F.Cu at (164.5, 77.0)
- moved LS3 42.5 mm to (142.0, 76.0), turned to 180 degrees
- moved LS1 42.4 mm to (142.0, 47.9)
- moved LS2 40.1 mm to (155.3, 47.5), turned to 180 degrees
- moved LS4 40.0 mm to (155.0, 76.0), turned to 180 degrees
- moved U1 0.20 mm to (147.6, 62.4)
Connections:
- LS1 pad 1: unconnected-(LS1-SS/-Pad1) -> Net-(LS1-SS/)
- LS1 pad 11: unconnected-(LS1-Ay-Pad11) -> Net-(C1-EncAy)
- LS1 pad 12: unconnected-(LS1-By-Pad12) -> Net-(C1-EncBy)
- LS1 pad 16: unconnected-(LS1-VDD-Pad16) -> Net-(C1-3v3)
- LS1 pad 2: unconnected-(LS1-SCK-Pad2) -> Net-(LS1-SCK)
- LS1 pad 3: unconnected-(LS1-MISO-Pad3) -> Net-(LS1-MISO)
- LS1 pad 4: unconnected-(LS1-MOSI-Pad4) -> Net-(LS1-MOSI)
- LS1 pad 5: unconnected-(LS1-Ax-Pad5) -> Net-(C1-EncAx)
- LS1 pad 6: unconnected-(LS1-Bx-Pad6) -> Net-(C1-EncBx)
- LS1 pad 8: unconnected-(LS1-GND-Pad8) -> Net-(C1-GND)
- LS2 pad 1: unconnected-(LS2-SS/-Pad1) -> Net-(LS2-SS/)
- LS2 pad 11: unconnected-(LS2-Ay-Pad11) -> Net-(C2-EncAy)
- LS2 pad 12: unconnected-(LS2-By-Pad12) -> Net-(C2-EncBy)
- LS2 pad 16: unconnected-(LS2-VDD-Pad16) -> Net-(C1-3v3)
- LS2 pad 2: unconnected-(LS2-SCK-Pad2) -> Net-(LS1-SCK)
- LS2 pad 3: unconnected-(LS2-MISO-Pad3) -> Net-(LS1-MISO)
- LS2 pad 4: unconnected-(LS2-MOSI-Pad4) -> Net-(LS1-MOSI)
- LS2 pad 5: unconnected-(LS2-Ax-Pad5) -> Net-(C2-EncAx)
- LS2 pad 6: unconnected-(LS2-Bx-Pad6) -> Net-(C2-DirBx)
- LS2 pad 8: unconnected-(LS2-GND-Pad8) -> Net-(C1-GND)
- LS3 pad 1: unconnected-(LS3-SS/-Pad1) -> Net-(LS3-SS/)
- LS3 pad 11: unconnected-(LS3-Ay-Pad11) -> Net-(C3-EncAy)
- LS3 pad 12: unconnected-(LS3-By-Pad12) -> Net-(C3-EncBy)
- LS3 pad 16: unconnected-(LS3-VDD-Pad16) -> Net-(C1-3v3)
- LS3 pad 2: unconnected-(LS3-SCK-Pad2) -> Net-(LS1-SCK)
- LS3 pad 3: unconnected-(LS3-MISO-Pad3) -> Net-(LS1-MISO)
- LS3 pad 4: unconnected-(LS3-MOSI-Pad4) -> Net-(LS1-MOSI)
- LS3 pad 5: unconnected-(LS3-Ax-Pad5) -> Net-(C3-EncAx)
- LS3 pad 6: unconnected-(LS3-Bx-Pad6) -> Net-(C3-EncBx)
- LS3 pad 8: unconnected-(LS3-GND-Pad8) -> Net-(C1-GND)
- LS4 pad 1: unconnected-(LS4-SS/-Pad1) -> Net-(LS4-SS/)
- LS4 pad 11: unconnected-(LS4-Ay-Pad11) -> Net-(C4-EncAy)
- LS4 pad 12: unconnected-(LS4-By-Pad12) -> Net-(C4-EncBy)
- LS4 pad 16: unconnected-(LS4-VDD-Pad16) -> Net-(C1-3v3)
- LS4 pad 2: unconnected-(LS4-SCK-Pad2) -> Net-(LS1-SCK)
- LS4 pad 3: unconnected-(LS4-MISO-Pad3) -> Net-(LS1-MISO)
- LS4 pad 4: unconnected-(LS4-MOSI-Pad4) -> Net-(LS1-MOSI)
- LS4 pad 5: unconnected-(LS4-Ax-Pad5) -> Net-(LS4-Ax)
- LS4 pad 6: unconnected-(LS4-Bx-Pad6) -> Net-(LS4-Bx)
- LS4 pad 8: unconnected-(LS4-GND-Pad8) -> Net-(C1-GND)
- U1 pad 13: unconnected-(U1-11_MOSI_CTX1-Pad13) -> Net-(LS1-MOSI)
- U1 pad 14: unconnected-(U1-12_MISO_MQSL-Pad14) -> Net-(LS1-MISO)
- U1 pad 15: unconnected-(U1-3V3-Pad15) -> Net-(C1-3v3)
- U1 pad 34: unconnected-(U1-GND-Pad34) -> Net-(C1-GND)
- U1 pad 35: unconnected-(U1-13_SCK_LED-Pad35) -> Net-(LS1-SCK)
- U1 pad 4: unconnected-(U1-2_OUT2-Pad4) -> Net-(LS1-SS/)
- U1 pad 5: unconnected-(U1-3_LRCLK2-Pad5) -> Net-(LS2-SS/)
- U1 pad 6: unconnected-(U1-4_BCLK2-Pad6) -> Net-(LS4-SS/)
- U1 pad 7: unconnected-(U1-5_IN2-Pad7) -> Net-(LS3-SS/)

Commit message: Final?
Parts:
- added J1: 5V in, Connector_Molex:Molex_Nano-Fit_105309-xx02_1x02_P2.50mm_Vertical, F.Cu at (113.5, 50.5)
- moved LS2 0.56 mm to (155.0, 48.0), turned to 0 degrees
- moved LS1 0.05 mm to (142.0, 48.0)
Connections:
- C1 pad 10: unconnected-(C1-DirBy-Pad10) -> Net-(C1-DirBy)
- C1 pad 2: unconnected-(C1-ENx-Pad2) -> Net-(C1-ENx)
- C1 pad 3: unconnected-(C1-DirAx-Pad3) -> Net-(C1-DirAx)
- C1 pad 4: unconnected-(C1-DirBx-Pad4) -> Net-(C1-DirBx)
- C1 pad 8: unconnected-(C1-ENy-Pad8) -> Net-(C1-ENy)
- C1 pad 9: unconnected-(C1-DirAy-Pad9) -> Net-(C1-DirAy)
- C2 pad 10: unconnected-(C2-DirBy-Pad10) -> Net-(C2-DirBy)
- C2 pad 2: unconnected-(C2-ENx-Pad2) -> Net-(C2-ENx)
- C2 pad 3: unconnected-(C2-DirAx-Pad3) -> Net-(C2-DirAx)
- C2 pad 6: unconnected-(C2-EncBx-Pad6) -> Net-(C2-EncBx)
- C2 pad 8: unconnected-(C2-ENy-Pad8) -> Net-(C2-ENy)
- C2 pad 9: unconnected-(C2-DirAy-Pad9) -> Net-(C2-DirAy)
- C3 pad 10: unconnected-(C3-DirBy-Pad10) -> Net-(C3-DirBy)
- C3 pad 2: unconnected-(C3-ENx-Pad2) -> Net-(C3-ENx)
- C3 pad 3: unconnected-(C3-DirAx-Pad3) -> Net-(C3-DirAx)
- C3 pad 4: unconnected-(C3-DirBx-Pad4) -> Net-(C3-DirBx)
- C3 pad 8: unconnected-(C3-ENy-Pad8) -> Net-(C3-ENy)
- C3 pad 9: unconnected-(C3-DirAy-Pad9) -> Net-(C3-DirAy)
- C4 pad 10: unconnected-(C4-DirBy-Pad10) -> Net-(C4-DirBy)
- C4 pad 2: unconnected-(C4-ENx-Pad2) -> Net-(C4-ENx)
- C4 pad 3: unconnected-(C4-DirAx-Pad3) -> Net-(C4-DirAx)
- C4 pad 4: unconnected-(C4-DirBx-Pad4) -> Net-(C4-DirBx)
- C4 pad 8: unconnected-(C4-ENy-Pad8) -> Net-(C4-ENy)
- C4 pad 9: unconnected-(C4-DirAy-Pad9) -> Net-(C4-DirAy)
- LS2 pad 6: Net-(C2-DirBx) -> Net-(C2-EncBx)
- U1 pad 10: unconnected-(U1-8_TX2_IN1-Pad10) -> Net-(C1-DirBy)
- U1 pad 16: unconnected-(U1-24_A10_TX6_SCL2-Pad16) -> Net-(C2-ENy)
- U1 pad 17: unconnected-(U1-25_A11_RX6_SDA2-Pad17) -> Net-(C2-DirAy)
- U1 pad 18: unconnected-(U1-26_A12_MOSI1-Pad18) -> Net-(C2-DirBy)
- U1 pad 19: unconnected-(U1-27_A13_SCK1-Pad19) -> Net-(C3-ENy)
- U1 pad 20: unconnected-(U1-28_RX7-Pad20) -> Net-(C3-DirAy)
- U1 pad 21: unconnected-(U1-29_TX7-Pad21) -> Net-(C3-DirBy)
- U1 pad 22: unconnected-(U1-30_CRX3-Pad22) -> Net-(C4-ENy)
- U1 pad 23: unconnected-(U1-31_CTX3-Pad23) -> Net-(C4-DirAy)
- U1 pad 24: unconnected-(U1-32_OUT1B-Pad24) -> Net-(C4-DirBy)
- U1 pad 30: unconnected-(U1-38_CS1_IN1-Pad30) -> Net-(C3-DirBx)
- U1 pad 31: unconnected-(U1-39_MISO1_OUT1A-Pad31) -> Net-(C4-DirBx)
- U1 pad 32: unconnected-(U1-40_A16-Pad32) -> Net-(C4-DirAx)
- U1 pad 33: unconnected-(U1-41_A17-Pad33) -> Net-(C4-ENx)
- U1 pad 38: unconnected-(U1-16_A2_RX4_SCL1-Pad38) -> Net-(C3-DirAx)
- U1 pad 39: unconnected-(U1-17_A3_TX4_SDA1-Pad39) -> Net-(C3-ENx)
- U1 pad 40: unconnected-(U1-18_A4_SDA-Pad40) -> Net-(C2-DirBx)
- U1 pad 41: unconnected-(U1-19_A5_SCL-Pad41) -> Net-(C2-DirAx)
- U1 pad 42: unconnected-(U1-20_A6_TX5_LRCLK1-Pad42) -> Net-(C2-ENx)
- U1 pad 43: unconnected-(U1-21_A7_RX5_BCLK1-Pad43) -> Net-(C1-DirBx)
- U1 pad 44: unconnected-(U1-22_A8_CTX1-Pad44) -> Net-(C1-DirAx)
- U1 pad 45: unconnected-(U1-23_A9_CRX1_MCLK1-Pad45) -> Net-(C1-ENx)
- U1 pad 47: unconnected-(U1-GND-Pad47) -> Net-(J1-Pin_1)
- U1 pad 48: unconnected-(U1-VIN-Pad48) -> Net-(J1-Pin_2)
- U1 pad 8: unconnected-(U1-6_OUT1D-Pad8) -> Net-(C1-ENy)
- U1 pad 9: unconnected-(U1-7_RX2_OUT1A-Pad9) -> Net-(C1-DirAy)
Routing:
- net Net-(C1-3v3): track 0.00 -> 173.4 mm
- net Net-(C1-GND): track 0.00 -> 156.6 mm, vias 0 -> 1
- net Net-(LS1-MOSI): track 0.00 -> 83.8 mm, vias 0 -> 4
- net Net-(LS1-SCK): track 0.00 -> 72.6 mm, vias 0 -> 5
- net Net-(LS1-MISO): track 0.00 -> 66.8 mm, vias 0 -> 3
- net Net-(LS2-SS/): track 0.00 -> 65.1 mm, vias 0 -> 1
- net Net-(C2-ENy): track 0.00 -> 62.8 mm
- net Net-(C2-DirAy): track 0.00 -> 61.4 mm
- net Net-(C2-DirBy): track 0.00 -> 59.8 mm
- net Net-(C4-ENx): track 0.00 -> 56.9 mm
- net Net-(C3-DirBx): track 0.00 -> 51.3 mm
- net Net-(C4-DirAx): track 0.00 -> 50.0 mm
- net Net-(C2-ENx): track 0.00 -> 47.2 mm
- net Net-(C3-DirBy): track 0.00 -> 44.5 mm
- net Net-(C3-DirAy): track 0.00 -> 44.5 mm
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Other:
- board outline added: 77 x 44 mm
- copper layers 2 -> 4
